File: drs-dev.kicad_pcb (KiCad board)
At the start: 2 copper layers, 58 x 58 mm, 58 parts, among them J1 Conn_01x03_Pin, J2 USB_C_Receptacle_USB2.0_16P, J3 Conn_ARM_SWD_TagConnect_TC203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, J4 Conn_01x03_Pin, J5 Conn_01x03_Pin, J6 Conn_01x03_Pin, J7 Barrel_Jack_Switch, U1 TPS5450DDAR, U2 TPS5450DDAR, U4 SRV05-4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

Commit message: Add labels and fix pinout
Connections:
- J1 pad 2: /PWM1 -> /PWR1
- J1 pad 3: /PWR1 -> /PWM1
- J4 pad 2: /PWM2 -> /PWR2
- J4 pad 3: /PWR2 -> /PWM2
Routing:
- net /PWR1: track 31.3 -> 38.6 mm, vias 11 -> 12
Other:
- board text added: "POS1"
- board text added: "POS2"
- board text added: "S+-"
