File: drs-dev.kicad_pcb (KiCad board)
At the start: 2 copper layers, 58 x 58 mm, 58 parts, among them J1 Conn_01x03_Pin, J2 USB_C_Receptacle_USB2.0_16P, J3 Conn_ARM_SWD_TagConnect_TC203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, J4 Conn_01x03_Pin, J5 Conn_01x03_Pin, J6 Conn_01x03_Pin, J7 Barrel_Jack_Switch, U1 TPS5450DDAR, U2 TPS5450DDAR, U4 SRV05-4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

Commit message: Fix usb pullup and generate new fab files
Parts:
- added R10: 1k5, Resistor_SMD:R_0402_1005Metric, F.Cu at (70.9, 68.3)
Routing:
- net +3V3: track 68.2 -> 73.1 mm
- net GND: track 87.5 -> 86.0 mm, vias 81 -> 83
